File: circuit/kicad/Esp8266-DomoticzAlarm-2B/Esp8266-DomoticzAlarm-2B.kicad_pcb (KiCad board)
At the start: 4 copper layers, 66 x 33.5 mm, 28 parts, among them J1 Barrel_Jack_Switch, Q1 BC817, Q2 BC817, U1 CH32V003JxMx, U2 ESP-12E, U4 MIC5219-3.3YM5

Commit message: circuit: power over HT7333. PDF. READ.md
Parts:
- added U3: HT7333, Package_TO_SOT_SMD:SOT-89-3, F.Cu at (131.5, 102.5)
- moved U4 3.77 mm to (125.7, 103.2)
Routing:
- net CH_VDD: track 98.7 -> 112.9 mm
- net CH_GND: track 182.1 -> 192.8 mm
- net B1+: track 109.3 -> 98.8 mm
- net Net-(U4-BP): track 2.25 -> 5.71 mm

Commit message: little changes in PCB
Parts:
- moved CH_C5 2.37 mm to (125.8, 98.7), turned to -90 degrees
Routing:
- net CH_GND: track 192.8 -> 188.1 mm
- net Net-(U4-BP): track 5.71 -> 3.20 mm
- net B1+: track 98.8 -> 100.3 mm
Other:
- board text added: "R260210"
- board text added: "T-AS260210"
- board text removed: "R251225"
Changed lines of the file:
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@@
 	(footprint "Capacitor_SMD:C_0805_2012Metric"
 		(layer "F.Cu")
-		(at 124.2 96.9)
+		(at 125.8 98.65 -90)
 		(descr "Capacitor SMD 0805 (2012 Metric), square (rectangular) end terminal, IPC-7351 nominal, (Body size source: IPC-SM-782 page 76, https://www.pcb-3d.com/wordpress/wp-content/uploads/ipc-sm-782a_amendment_1_and_2.pdf, https://docs.google.com/spreadsheets/d/1BsfQQcO9C6DZCsRaXUlFlo91Tg2WpOkGARC1WS5S8t0/edit?usp=sharing), generated with kicad-footprint-generator")
 		(tags "capacitor")
 		(property "Reference" "CH_C5"
-			(at 0 -1.68 0)
+			(at 0 -1.68 90)
 			(layer "F.SilkS")
 			(hide yes)
@@
 		)
 		(property "Value" "470nF"
-			(at 0 1.68 0)
+			(at 0 1.68 90)
 			(layer "F.Fab")
 			(hide yes)
@@
 		)
 		(property "Datasheet" "~"
-			(at 0 0 0)
+			(at 0 0 90)
 			(layer "F.Fab")
 			(hide yes)
@@
 		)
 		(property "Description" "Unpolarized capacitor"
-			(at 0 0 0)
+			(at 0 0 90)
 			(layer "F.Fab")
 			(hide yes)
@@
 		(attr smd)
 		(fp_line
-			(start -0.261252 -0.735)
-			(end 0.261252 -0.735)
+			(start -0.261252 0.735)
+			(end 0.261252 0.735)
 			(stroke
 				(width 0.12)
@@
 		)
 		(fp_line
-			(start -0.261252 0.735)
-			(end 0.261252 0.735)
+			(start -0.261252 -0.735)
+			(end 0.261252 -0.735)
 			(stroke
 				(width 0.12)
@@
 		)
 		(fp_line
-			(start -1.7 -0.98)
-			(end 1.7 -0.98)
+			(start -1.7 0.98)
+			(end -1.7 -0.98)
 			(stroke
 				(width 0.05)
@@
 		)
 		(fp_line
-			(start -1.7 0.98)
-			(end -1.7 -0.98)
+			(start 1.7 0.98)
+			(end -1.7 0.98)
 			(stroke
 				(width 0.05)
@@
 		)
 		(fp_line
-			(start 1.7 -0.98)
-			(end 1.7 0.98)
+			(start -1.7 -0.98)
+			(end 1.7 -0.98)
 			(stroke
 				(width 0.05)
@@
 		)
 		(fp_line
-			(start 1.7 0.98)
-			(end -1.7 0.98)
+			(start 1.7 -0.98)
+			(end 1.7 0.98)
 			(stroke
 				(width 0.05)
@@
 		)
 		(fp_line
-			(start -1 -0.625)
-			(end 1 -0.625)
+			(start -1 0.625)
+			(end -1 -0.625)
 			(stroke
 				(width 0.1)
@@
 		)
 		(fp_line
-			(start -1 0.625)
-			(end -1 -0.625)
+			(start 1 0.625)
+			(end -1 0.625)
 			(stroke
 				(width 0.1)
@@
 		)
 		(fp_line
-			(start 1 -0.625)
-			(end 1 0.625)
+			(start -1 -0.625)
+			(end 1 -0.625)
 			(stroke
 				(width 0.1)
@@
 		)
 		(fp_line
-			(start 1 0.625)
-			(end -1 0.625)
+			(start 1 -0.625)
+			(end 1 0.625)
 			(stroke
 				(width 0.1)
@@
 		)
 		(fp_text user "${REFERENCE}"
-			(at 0 0 0)
+			(at 0 0 90)
 			(layer "F.Fab")
 			(effects
@@
 		)
 		(pad "1" smd roundrect
-			(at -0.95 0)
+			(at -0.95 0 270)
 			(size 1 1.45)
 			(layers "F.Cu" "F.Mask" "F.Paste")
@@
 		)
 		(pad "2" smd roundrect
-			(at 0.95 0)
+			(at 0.95 0 270)
 			(size 1 1.45)
 			(layers "F.Cu" "F.Mask" "F.Paste")
@@
 		(layer "Edge.Cuts")
 	)
-	(gr_text "T-AS251211"
+	(gr_text "T-AS260210"
 		(at 81.1 92.1 0)
 		(layer "F.Cu")
@@
 		)
 	)
-	(gr_text "T-AS251211"
+	(gr_text "T-AS260210"
 		(at 92.6 92.1 0)
 		(layer "B.Cu")
@@
 		)
 	)
-	(gr_text "R251225"
+	(gr_text "R260210"
 		(at 81 94.1 0)
 		(layer "F.SilkS")
@@
 		)
 	)
-	(gr_text "R251225"
+	(gr_text "R260210"
 		(at 81 92.9 180)
 		(layer "B.SilkS")
@@
 	)
 	(segment
-		(start 86.2 120.4)
-		(end 86.5 120.1)
+		(start 127.3 97.7)
+		(end 129.55 99.95)
 		(width 0.5)
 		(layer "F.Cu")
@@
 	)
 	(segment
-		(start 125.8 102.8)
-		(end 125.8 101.7)
+		(start 86.2 120.4)
+		(end 86.5 120.1)
 		(width 0.5)
 		(layer "F.Cu")
@@
 	)
 	(segment
-		(start 123.5 98.85)
-		(end 123.5 97.15)
+		(start 125.8 102.8)
+		(end 125.8 101.7)
 		(width 0.5)
 		(layer "F.Cu")
@@
 	)
 	(segment
-		(start 126.4 95.4)
-		(end 129.55 98.55)
+		(start 123.5 98.85)
+		(end 124.65 97.7)
 		(width 0.5)
 		(layer "F.Cu")
@@
 	)
 	(segment
+		(start 124.65 97.7)
+		(end 125.8 97.7)
+		(width 0.5)
+		(layer "F.Cu")
+		(net 1)
+	)
+	(segment
 		(start 86.823 98.386)
 		(end 86.723 98.486)
@@
 	)
 	(segment
-		(start 123.25 96.9)
-		(end 123.3 96)
+		(start 85.423 106.186)
+		(end 86.823 104.786)
 		(width 0.5)
 		(layer "F.Cu")
@@
 	)
 	(segment
-		(start 123.9 95.4)
-		(end 126.4 95.4)
+		(start 79 110.484)
+		(end 79 118.6)
 		(width 0.5)
 		(layer "F.Cu")
@@
 	)
 	(segment
-		(start 85.423 106.186)
-		(end 86.823 104.786)
+		(start 80.772 108.712)
+		(end 79 110.484)
 		(width 0.5)
 		(layer "F.Cu")
@@
 	)
 	(segment
-		(start 79 110.484)
-		(end 79 118.6)
+		(start 125.8 97.7)
+		(end 127.3 97.7)
 		(width 0.5)
 		(layer "F.Cu")
@@
 	)
 	(segment
-		(start 129.55 98.55)
+		(start 129.55 99.95)
 		(end 129.55 101)
 		(width 0.5)
@@
 	)
 	(segment
-		(start 80.772 108.712)
-		(end 79 110.484)
-		(width 0.5)
-		(layer "F.Cu")
-		(net 1)
-	)
-	(segment
 		(start 116.84 112.172)
 		(end 116.953 112.059)
@@
 	)
 	(segment
-		(start 123.5 97.15)
-		(end 123.25 96.9)
-		(width 0.5)
-		(layer "F.Cu")
-		(net 1)
-	)
-	(segment
-		(start 123.3 96)
-		(end 123.9 95.4)
-		(width 0.5)
-		(layer "F.Cu")
-		(net 1)
-	)
-	(segment
 		(start 79 118.6)
 		(end 79 119.8)
@@
 	)
 	(segment
+		(start 125.65 105.425)
+		(end 126.875 104.2)
+		(width 0.5)
+		(layer "F.Cu")
+		(net 7)
+	)
+	(segment
 		(start 126.875 102.3)
 		(end 128.2 102.3)
@@
 	)
 	(segment
+		(start 125.65 106.15)
+		(end 125.65 105.425)
+		(width 0.5)
+		(layer "F.Cu")
+		(net 7)
+	)
+	(segment
 		(start 128.6 102.3)
 		(end 129.6375 102.5)
@@
 	(segment
 		(start 127.5 107.3)
-		(end 127.5 104.825)
+		(end 126.8 107.3)
 		(width 0.5)
 		(layer "F.Cu")
@@
 	)
 	(segment
-		(start 127.5 104.825)
-		(end 126.875 104.2)
+		(start 75.123 108.986)
+		(end 75.418 109.281)
 		(width 0.5)
 		(layer "F.Cu")
@@
 	)
 	(segment
-		(start 75.123 108.986)
-		(end 75.418 109.281)
+		(start 126.8 107.3)
+		(end 125.65 106.15)
 		(width 0.5)
 		(layer "F.Cu")
@@
 	)
 	(segment
-		(start 125.15 96.9)
-		(end 125.25 97)
+		(start 124.75 101.3)
+		(end 125.8 100.25)
 		(width 0.5)
 		(layer "F.Cu")
@@
 	)
 	(segment
-		(start 125.25 97)
-		(end 125.25 100.05)
-		(width 0.5)
-		(layer "F.Cu")
-		(net 31)
-	)
-	(segment
-		(start 125.25 100.05)
-		(end 124.75 100.55)
+		(start 124.6 102.3)
+		(end 124.75 102.15)
 		(width 0.5)
 		(layer "F.Cu")
@@
 	)
 	(segment
-		(start 124.75 100.55)
-		(end 124.75 102.15)
+		(start 125.8 100.25)
+		(end 125.8 99.6)
 		(width 0.5)
 		(layer "F.Cu")
@@
 	(segment
 		(start 124.75 102.15)
-		(end 124.6 102.3)
+		(end 124.75 101.3)
 		(width 0.5)
 		(layer "F.Cu")

Commit message: changes 20260416
Parts:
- removed CH_J1: Conn_01x04, Connector_PinHeader_2.54mm:PinHeader_1x04_P2.54mm_Vertical
- removed CH_J2: ~, Connector_PinHeader_2.54mm:PinHeader_1x04_P2.54mm_Vertical
- added D2: 1N5819WS, Diode_SMD:D_SOD-323_HandSoldering, F.Cu at (123.8, 118.9)
- CH_C2, CH_C4: footprint Capacitor_SMD:C_0805_2012Metric -> Capacitor_SMD:C_1206_3216Metric
- moved CH_C2 0.50 mm to (123.2, 99.4)
- moved CH_J7 0.35 mm to (79.0, 118.9)
Connections:
- J1 pad 1: CH_GND -> Net-(D2-A)
- J1 pad 2: B1+ -> CH_GND
- J1 pad 3: B1+ -> CH_GND
Routing:
- net CH_GND: track 188.1 -> 211.3 mm, vias 2 -> 1
- net ALARMFROMESP: track 33.6 -> 16.1 mm
- net ALARM_CAM_DI: track 34.7 -> 18.1 mm, vias 0 -> 1
- net CH_VDD: track 112.9 -> 101.9 mm, vias 0 -> 1
- net Net-(D2-A): track 0.00 -> 7.13 mm
- net CH_ALARM_BREAKE_A: track 25.2 -> 19.5 mm, vias 1 -> 2
- net SWITCH_ALARMSTATUS: track 10.3 -> 6.07 mm
- net CH_C4: track 44.3 -> 43.1 mm, vias 0 -> 1
- net B1+: track 100.3 -> 99.5 mm, vias 0 -> 2
Other:
- board text added: "R260404"
- board text added: "T-AS260404"
- board text removed: "R260210"
- board text removed: "T-AS260210"
