File: circuit/kicad/Esp8266-DomoticzAlarm-2B/Esp8266-DomoticzAlarm-2B.kicad_pcb (KiCad board)
At the start: 4 copper layers, 66 x 33.5 mm, 28 parts, among them J1 Barrel_Jack_Switch, Q1 BC817, Q2 BC817, U1 CH32V003JxMx, U2 ESP-12E, U3 HT7333, U4 MIC5219-3.3YM5

Commit message: KiCAD changes for ver 261026 The Siren-connector have new one connection over XH-2.50-H connector (2a)
Parts:
- added J2a1: Conn_01x02, Connector_JST:JST_XH_S2B-XH-A_1x02_P2.50mm_Horizontal, F.Cu at (94.3, 112.6)
Routing:
- net CH_ALARM_IN: track 11.8 -> 31.6 mm
- net CH_GND: track 211.3 -> 214.6 mm
- net CH_VDD: track 101.9 -> 101.3 mm
Other:
- board text added: "R261026"
- board text added: "T-AS261026"
- board text removed: "R260404"
- board text removed: "T-AS251211"
